File: swinsid.sch (KiCad schematic (older format))
At the start: 14 parts, among them J1 Conn_PIC_ICSP_ICD, U1 ATmega88PA-AU, U2 SID6581, X1 SG-7050CAN

Commit message: Updated swinsid image
Parts:
- added SW1: SW_DIP_x02, Button_Switch_SMD:SW_DIP_SPSTx02_Slide_9.78x7.26mm_W8.61mm_P2.54mm, symbol Switch:SW_DIP_x02
Changed lines of the file:
@@
 Wire Wire Line
 	1300 5200 1150 5200
+$Comp
+L Switch:SW_DIP_x02 SW1
+U 1 1 613DFD45
+P 7750 3600
+F 0 "SW1" H 7750 3967 50  0000 C CNN
+F 1 "SW_DIP_x02" H 7750 3876 50  0000 C CNN
+F 2 "Button_Switch_SMD:SW_DIP_SPSTx02_Slide_9.78x7.26mm_W8.61mm_P2.54mm" H 7750 3600 50  0001 C CNN
+F 3 "~" H 7750 3600 50  0001 C CNN
+	1    7750 3600
+	1    0    0    -1
+$EndComp
 $EndSCHEMATC
